Commit message: Add linetrace_code

File: urdf/cp.urdf (robot description, URDF)
Before this commit: robot wheel_robot_simple, 13 links, 12 joints
Links:
- removed link linetrace_link2
- removed link linetrace_link3
- removed link linetrace_link4
- removed link linetrace_link5
- link back_ball_link: mass 0.095 -> 0.03; geometry collision sphere radius=0.015; visual sphere radius=0.015
- link body_link: mass 0.7 -> 1.0
- link camera_link: mass 0.070 -> 0.1
- link elbow_link: mass 0.220 -> 0.08
- link left_wheel_link: mass 0.120 -> 0.2; geometry collision cylinder length=0.04 radius=0.036; visual cylinder length=0.04 radius=0.036
- link right_wheel_link: mass 0.120 -> 0.2; geometry collision cylinder length=0.04 radius=0.036; visual cylinder length=0.04 radius=0.036
- link sholder_base_link: mass 0.060 -> 0.06
- link sholder_link: mass 0.060 -> 0.08
Joints:
- removed joint linetrace_joint2
- removed joint linetrace_joint3
- removed joint linetrace_joint4
- removed joint linetrace_joint5
- joint back_ball_joint: origin xyz=-0.13 0.0 0.0 rpy=0.0 0.0 0.0 -> xyz=-0.13 0.0 -0.022 rpy=0.0 0.0 0.0
- joint body_joint: origin xyz=-0.6 -0.8 0.4 rpy=0.0 0.0 1.5708 -> xyz=-0.3 0.0 0.2 rpy=0.0 0.0 -1.5708
- joint camera_joint: origin xyz=0.13 0 0.01 rpy=0 0 0 -> xyz=0.15 0 0.01 rpy=0 0 0
