Commit message: Add file

File: urdf/wheel_robot_simple.urdf (robot description, URDF)
Before this commit: robot wheel_robot_simple, 13 links, 12 joints
Links:
- removed link back_ball_link
- added link box_link1, mass 0.14664217699835314; collision mesh filename=file:///home/ikenta/ros2_ws/src/arm_detecting_controll/mode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 scale=0.001 0.001 0.001; visual mesh filename=file:///home/ikenta/ros2_ws/src/arm_detecting_controll/mode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 scale=0.001 0.001 0.001
- added link box_link2, mass 0.14664217699835314; collision mesh filename=file:///home/ikenta/ros2_ws/src/arm_detecting_controll/mode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 scale=0.001 0.001 0.001; visual mesh filename=file:///home/ikenta/ros2_ws/src/arm_detecting_controll/mode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 scale=0.001 0.001 0.001
- added link box_link3, mass 0.14664217699835314; collision mesh filename=file:///home/ikenta/ros2_ws/src/arm_detecting_controll/mode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 scale=0.001 0.001 0.001; visual mesh filename=file:///home/ikenta/ros2_ws/src/arm_detecting_controll/mode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 scale=0.001 0.001 0.001
- added link camera_link1, mass 0.0001; collision box size=0.0002 0.0002 0.0002; visual box size=0.0002 0.0002 0.0002
- added link camera_stopper_link, mass 0.0132681554963914; collision mesh filename=file:///home/ikenta/ros2_ws/src/arm_detecting_controll/mode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 scale=0.001 0.001 0.001; visual mesh filename=file:///home/ikenta/ros2_ws/src/arm_detecting_controll/mode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 scale=0.001 0.001 0.001
- added link castor_link, mass 0.03; collision mesh filename=file:///home/ikenta/ros2_ws/src/arm_detecting_controll/mode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 scale=0.001 0.001 0.001; visual mesh filename=file:///home/ikenta/ros2_ws/src/arm_detecting_controll/mode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 scale=0.001 0.001 0.001
- added link fan_link, mass 0.019203927572863683; collision mesh filename=file:///home/ikenta/ros2_ws/src/arm_detecting_controll/mode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 scale=0.001 0.001 0.001; visual mesh filename=file:///home/ikenta/ros2_ws/src/arm_detecting_controll/mode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 scale=0.001 0.001 0.001
- added link fancase_link, mass 0.029214118817680147; collision mesh filename=file:///home/ikenta/ros2_ws/src/arm_detecting_controll/mode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 scale=0.001 0.001 0.001; visual mesh filename=file:///home/ikenta/ros2_ws/src/arm_detecting_controll/mode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 scale=0.001 0.001 0.001
- added link left_motor_link, mass 0.12809503672651354; collision mesh filename=file:///home/ikenta/ros2_ws/src/arm_detecting_controll/mode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 scale=0.001 0.001 0.001; visual mesh filename=file:///home/ikenta/ros2_ws/src/arm_detecting_controll/mode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 scale=0.001 0.001 0.001
- added link linetrace_link, mass 0.005248538060524059; collision mesh filename=file:///home/ikenta/ros2_ws/src/arm_detecting_controll/mode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 scale=0.001 0.001 0.001; visual mesh filename=file:///home/ikenta/ros2_ws/src/arm_detecting_controll/mode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 scale=0.001 0.001 0.001
- added link prop_link1, mass 0.04116435399670614; collision mesh filename=file:///home/ikenta/ros2_ws/src/arm_detecting_controll/mode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 scale=0.001 0.001 0.001; visual mesh filename=file:///home/ikenta/ros2_ws/src/arm_detecting_controll/mode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 scale=0.001 0.001 0.001
- added link prop_link2, mass 0.04116435399670614; collision mesh filename=file:///home/ikenta/ros2_ws/src/arm_detecting_controll/mode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 scale=0.001 0.001 0.001; visual mesh filename=file:///home/ikenta/ros2_ws/src/arm_detecting_controll/mode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 scale=0.001 0.001 0.001
- added link prop_link3, mass 0.04116435399670614; collision mesh filename=file:///home/ikenta/ros2_ws/src/arm_detecting_controll/mode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 scale=0.001 0.001 0.001; visual mesh filename=file:///home/ikenta/ros2_ws/src/arm_detecting_controll/mode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 scale=0.001 0.001 0.001
- added link right_motor_link, mass 0.12809503672651354; collision mesh filename=file:///home/ikenta/ros2_ws/src/arm_detecting_controll/mode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 scale=0.001 0.001 0.001; visual mesh filename=file:///home/ikenta/ros2_ws/src/arm_detecting_controll/mode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 scale=0.001 0.001 0.001
- added link spacer_link1, mass 0.0014886724402471767; collision mesh filename=file:///home/ikenta/ros2_ws/src/arm_detecting_controll/mode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 scale=0.001 0.001 0.001; visual mesh filename=file:///home/ikenta/ros2_ws/src/arm_detecting_controll/mode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 scale=0.001 0.001 0.001
- added link spacer_link2, mass 0.0014886724402471767; collision mesh filename=file:///home/ikenta/ros2_ws/src/arm_detecting_controll/mode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 scale=0.001 0.001 0.001; visual mesh filename=file:///home/ikenta/ros2_ws/src/arm_detecting_controll/mode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 scale=0.001 0.001 0.001
- link body_link: mass 0.7 -> 0.21361792130545304; geometry collision mesh filename=file:///home/ikenta/ros2_ws/src/arm_detecting_controll/mode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 scale=0.001 0.001 0.001; visual mesh filename=file:///home/ikenta/ros2_ws/src/arm_detecting_controll/mode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 scale=0.001 0.001 0.001
- link camera_link: mass 0.070 -> 0.06369938289373575; geometry collision mesh filename=file:///home/ikenta/ros2_ws/src/arm_detecting_controll/mode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 scale=0.001 0.001 0.001; visual mesh filename=file:///home/ikenta/ros2_ws/src/arm_detecting_controll/mode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 scale=0.001 0.001 0.001
- link elbow_link: mass 0.220 -> 0.10768771500759752; geometry collision mesh filename=file:///home/ikenta/ros2_ws/src/arm_detecting_controll/mode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 scale=0.001 0.001 0.001; visual mesh filename=file:///home/ikenta/ros2_ws/src/arm_detecting_controll/mode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 scale=0.001 0.001 0.001
- link left_wheel_link: mass 0.120 -> 0.2; geometry collision cylinder length=0.003 radius=0.0255; visual cylinder length=0.003 radius=0.0255
- link right_wheel_link: mass 0.120 -> 0.2; geometry collision cylinder length=0.003 radius=0.0255; visual cylinder length=0.003 radius=0.0255
- link sholder_base_link: mass 0.060 -> 0.04805535665511946; geometry collision mesh filename=file:///home/ikenta/ros2_ws/src/arm_detecting_controll/mode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 scale=0.001 0.001 0.001; visual mesh filename=file:///home/ikenta/ros2_ws/src/arm_detecting_controll/mode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 scale=0.001 0.001 0.001
- link sholder_link: mass 0.060 -> 0.11107447123195605; geometry collision mesh filename=file:///home/ikenta/ros2_ws/src/arm_detecting_controll/mode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 scale=0.001 0.001 0.001; visual mesh filename=file:///home/ikenta/ros2_ws/src/arm_detecting_controll/mode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 scale=0.001 0.001 0.001
Joints:
- removed joint back_ball_joint
- removed joint elbow_arm
- removed joint sholder_arm
- added joint box_joint1: type fixed, parent prop_link1, child box_link1, origin xyz=0.081 -0.073 0.078 rpy=0 0 0
- added joint box_joint2: type fixed, parent prop_link2, child box_link2, origin xyz=0.084 0.209 0.166 rpy=0 1.5708 0
- added joint box_joint3: type fixed, parent prop_link3, child box_link3, origin xyz=0.081 -0.073 0.078 rpy=0 0 0
- added joint camera_joint1: type fixed, parent camera_link, child camera_link1, origin xyz=-0.047 0.019 0.006 rpy=0 0 3.1416
- added joint camera_stopper_joint: type fixed, parent body_link, child camera_stopper_link, origin xyz=0.093 0.0815 0.0 rpy=0 0 0
- added joint castor_joint: type fixed, parent body_link, child castor_link, origin xyz=0.336 0.1365 0.0 rpy=0 3.1416 3.1416
- added joint elbow_joint: type revolute, parent sholder_link, child elbow_link, origin xyz=5e-06 -0.0255 0.090232 rpy=0 0 0, axis 0.0 -1.0 -0.0, limit lower=-0.872665 upper=2.181662 effort=100 velocity=100
- added joint fan_joint: type fixed, parent fancase_link, child fan_link, origin xyz=0.0 0.0 0.003 rpy=0 0 0
- added joint fancase_joint: type fixed, parent elbow_link, child fancase_link, origin xyz=0.0 0.0255 0.178 rpy=0 0 0
- added joint left_motor_joint: type fixed, parent body_link, child left_motor_link, origin xyz=0.097 0.025 0.0 rpy=0 0 0
- added joint linetrace_joint: type fixed, parent spacer_link2, child linetrace_link, origin xyz=0.0 0.0 -0.043 rpy=0 0 0
- added joint prop_joint1: type fixed, parent body_link, child prop_link1, origin xyz=0.206 0.078 0.003 rpy=0 0 0
- added joint prop_joint2: type fixed, parent body_link, child prop_link2, origin xyz=0.206 0.161 0.003 rpy=0 0 0
- added joint prop_joint3: type fixed, parent body_link, child prop_link3, origin xyz=0.206 0.244 0.003 rpy=0 0 0
- added joint right_motor_joint: type fixed, parent body_link, child right_motor_link, origin xyz=0.097 0.224 0.0 rpy=0 0 0
- added joint sholder_base_joint: type fixed, parent body_link, child sholder_base_link, origin xyz=0.188 0.1195 0.003 rpy=0 0 0
- added joint spacer_joint1: type fixed, parent body_link, child spacer_link1, origin xyz=0.0875 0.0745 0.0 rpy=0 0 0
- added joint spacer_joint2: type fixed, parent body_link, child spacer_link2, origin xyz=0.0875 0.1745 0.0 rpy=0 0 0
- joint body_joint: origin xyz=-0.6 -0.8 0.4 rpy=0.0 0.0 1.5708 -> xyz=-0.7 -0.6 0.9 rpy=0.0 0.0 -1.5708
- joint camera_joint: origin xyz=0.13 0 0.01 rpy=0 0 0 -> xyz=0.01 0.023 -0.015 rpy=0 0 0; parent body_link -> camera_stopper_link
- joint left_wheel_joint: axis 0.0 0.0 1.0 -> -0.0 -0.0 1.0; origin xyz=0.1 0.1 -0.0 rpy=-1.5707 0.0 0.0 -> xyz=0.0 -0.045 -0.021 rpy=1.5708 0 0; parent body_link -> left_motor_link
- joint linetrace_joint2: origin xyz=0.125 0.024 -0.015 rpy=0 1.5708 0 -> xyz=-0.01 -0.074 -0.002 rpy=0 1.5708 0; parent body_link -> linetrace_link
- joint linetrace_joint3: origin xyz=0.125 0.008 -0.015 rpy=0 1.5708 0 -> xyz=-0.01 -0.058 -0.002 rpy=0 1.5708 0; parent body_link -> linetrace_link
- joint linetrace_joint4: origin xyz=0.125 -0.008 -0.015 rpy=0 1.5708 0 -> xyz=-0.01 -0.042 -0.002 rpy=0 1.5708 0; parent body_link -> linetrace_link
- joint linetrace_joint5: origin xyz=0.125 -0.024 -0.015 rpy=0 1.5708 0 -> xyz=-0.01 -0.026 -0.002 rpy=0 1.5708 0; parent body_link -> linetrace_link
- joint right_wheel_joint: axis 0.0 0.0 -1.0 -> 0.0 -0.0 1.0; origin xyz=0.1 -0.1 -0.0 rpy=1.5707 0.0 0.0 -> xyz=0.0 0.045 -0.021 rpy=1.5708 0 0; parent body_link -> right_motor_link
- joint sholder_joint: axis (none) -> -0.0 -0.0 -1.0; child sholder_base_link -> sholder_link; limit (none) -> lower=-1.047198 upper=1.047198 effort=100 velocity=100; origin xyz=0 0 0.01 rpy=0.0 0.0 -1.5708 -> xyz=-0.060732 0.005005 0.013 rpy=0 0 0; parent body_link -> sholder_base_link; type fixed -> revolute
