Commit message: Edit README

File: urdf/vacuum_robot.urdf (robot description, URDF)
Before this commit: robot wheel_robot_simple, 22 links, 21 joints
Joints:
- joint body_joint: origin xyz=0.6 0.4 0.4 rpy=0.0 0.0 -1.5708 -> xyz=-0.6 -0.7 0.4 rpy=0.0 0.0 -1.5708

Commit message: Edit files

File: urdf/vacuum_robot.urdf (robot description, URDF)
Before this commit: robot wheel_robot_simple, 22 links, 21 joints
Joints:
- joint body_joint: origin xyz=-0.6 -0.7 0.4 rpy=0.0 0.0 -1.5708 -> xyz=-0.6 -0.4 0.4 rpy=0.0 0.0 1.5708
